File: mainboard/mainboard.kicad_sch (KiCad schematic)
At the start: 81 parts, among them J1 USB_C_Receptacle_USB2.0_16P, J10 Barrel_Jack, J2 Conn_01x03_Pin, J4 Conn_01x04_Socket, J5 Conn_01x04_Socket, J6 Screw_Terminal_01x02, J7 Conn_01x02_Socket, J8 Conn_01x02_Socket, J9 Conn_01x04_Socket, Q1 BTN8982TA, Q2 AO3400A, Q3 AO3400A, Q6 BTN8982TA, U1 ESP32-S3-WROOM-1, U2 USBLC6-2SC6, U3 AP2112K-3.3, U4 TPS2116DRL, U5 TPS62161DSG

Commit message: worked on loadswitch layout, linear regulator layout
Parts:
- removed J10: Barrel_Jack, Connector_BarrelJack:BarrelJack_Wuerth_694108106102_2.5x5.5mm, symbol Connector:Barrel_Jack
- added J3: Barrel_Jack_MountingPin, Connector_BarrelJack:BarrelJack_Horizontal, symbol Connector:Barrel_Jack_MountingPin
- added R22: 10k, Resistor_SMD:R_0603_1608Metric, symbol Device:R
- R15: value 10k -> 52k3
Connections:
- net +12V: no longer F2.1
- net +5V: now also U5.6 (VOS)
- net GND: now also J3.2, J3.MP (MountPin), R22.2; no longer U5.8 (PG)
- net PR1: now reaches R17.1, U4.4 (PR1)
- net PR1: now also R22.1
- net FB: now reaches R15.1, R6.2, U5.5 (FB)
- net 5V_SEL: now reaches C4.1, U3.1 (VIN), U3.3 (EN), U4.2 (VOUT), U4.7 (VOUT)
- net SW: now reaches L2.1, U5.7 (SW)
- net SW: no longer U5.6 (VOS)
- net EN: now reaches R16.2, U5.3 (EN)
- new net 12V: F2.1, J3.1
- no-connect marks 18 -> 19
