File: hardware/sensor/sensor/sensor.kicad_sch (KiCad schematic)
At the start: 0 parts

Commit message: sensor footprint added, started schematic connections between the ESP and the sensors
Parts:
- added C1, C2: 1µ, symbol Device:C
- added C3: 100n, symbol Device:C
- added R: 4.7, symbol Device:R
- added R1, R2, Rp (x2): 10k, symbol Device:R
- added U1: SHT4x, Sensor_Humidity:Sensirion_DFN-4_1.5x1.5mm_P0.8mm_SHT4x_NoCentralPad, symbol Sensor_Humidity:SHT4x
- added U2: ESP32-C3-WROOM-02, RF_Module:ESP32-C3-WROOM-02, symbol RF_Module:ESP32-C3-WROOM-02
- added U3: AP2112K-3.3, Package_TO_SOT_SMD:SOT-23-5, symbol Regulator_Linear:AP2112K-3.3
- added U4: SGP40, symbol SGP40:SGP40
Connections:
- new net: R2.2, U1.1 (SDA), U2.6 (IO7)
- new net: C2.1, R.1, Rp.1, Rp.1, U4. (n/a)
- new net: Rp.2, U4. (n/a) (x2)
- new net: R1.2, U1.2 (SCL), U2.4 (IO5)
- new net: C1.1, R.2, U4. (n/a)
- new net: U3.1 (VIN), U3.3 (EN)
- new net +3.3V: C3.1, R1.1, R2.1, U1.3 (VDD), U2.1 (3V3)
- new net GND: C1.2, C2.2, C3.2, U2.19 (GND), U2.9 (GND), U3.2 (GND), U4. (n/a)
