File: hardware/mainboard/mainboard.kicad_pcb (KiCad board)
At the start: 4 copper layers, 101.9 x 66.3 mm, 92 parts, among them J1 USB_C_Receptacle_USB2.0_16P, J2 Conn_01x03_Pin, J3 Barrel_Jack_MountingPin, J4 Conn_01x04_Socket, J5 Conn_01x04_Socket, J6 Screw_Terminal_01x02, J7 Conn_01x02_Socket, J8 Conn_01x02_Socket, J9 Conn_01x04_Socket, Q1 BTN8982TA, Q2 AO3400A, Q3 AO3400A, Q4 AO3400A, Q5 AO3400A, Q6 BTN8982TA, U1 ESP32-S3-WROOM-1, U2 USBLC6-2SC6, U3 AP2112K-3.3, U4 TPS2116DRL, U5 TPS62161DSG

Commit message: small adjustments to timelog and docs
Parts:
- moved J9 7.62 mm to (193.7, 88.6), turned to -90 degrees
Routing:
- net SDA: track 45.1 -> 51.6 mm, vias 1 -> 2
- net SCL: track 49.3 -> 51.3 mm
Changed lines of the file:
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@@
 		)
 		(embedded_fonts no)
-		(model "${KICAD9_3DMODEL_DIR}/Fuse.3dshapes/Fuse_Littelfuse-NANO2-451_453.step"
+		(model "${KICAD9_3RD_PARTY}/045106.3MRL.STEP"
 			(offset
-				(xyz 0 0 0)
-			)
-			(scale
-				(xyz 1 1 1)
-			)
-			(rotate
-				(xyz 0 0 0)
-			)
-		)
-		(model "${KICAD9_3DMODEL_DIR}/Fuse.3dshapes/Fuse_1210_3225Metric.wrl"
-			(hide yes)
-			(offset
-				(xyz 0 0 0)
+				(xyz 0 -1.5 0)
 			)
 			(scale
@@
 			)
 			(rotate
-				(xyz 0 0 0)
-			)
-		)
-		(model "${KICAD9_3DMODEL_DIR}/Resistor_SMD.3dshapes/R_1806_4516Metric.step"
-			(hide yes)
-			(offset
-				(xyz 0 0 0)
-			)
-			(scale
-				(xyz 1 1 1)
-			)
-			(rotate
-				(xyz 0 0 0)
-			)
-		)
-		(model "${KICAD9_3DMODEL_DIR}/Resistor_SMD.3dshapes/R_2010_5025Metric.step"
-			(offset
-				(xyz 0 0 0)
-			)
-			(scale
-				(xyz 1 1 1)
-			)
-			(rotate
-				(xyz 0 0 0)
+				(xyz -0 -0 -0)
 			)
 		)
@@
 	(footprint "Connector_PinSocket_2.54mm:PinSocket_1x04_P2.54mm_Vertical"
 		(layer "F.Cu")
-		(at 186.075 88.575 90)
+		(at 193.7 88.575 -90)
 		(descr "Through hole straight socket strip, 1x04, 2.54mm pitch, single row (from Kicad 4.0.7), script generated")
 		(tags "Through hole socket strip THT 1x04 2.54mm single row")
 		(property "Reference" "J9"
-			(at -0.025 -2.82 180)
+			(at -0.025 -2.82 0)
 			(layer "F.SilkS")
 			(effects
@@
 		(attr through_hole)
 		(fp_line
-			(start 1.33 -1.33)
-			(end 1.33 0)
+			(start -1.33 8.95)
+			(end 1.33 8.95)
 			(stroke
 				(width 0.12)
@@
 		)
 		(fp_line
-			(start 0 -1.33)
-			(end 1.33 -1.33)
+			(start -1.33 1.27)
+			(end -1.33 8.95)
 			(stroke
 				(width 0.12)
@@
 		)
 		(fp_line
-			(start 1.33 1.27)
-			(end 1.33 8.95)
+			(start -1.33 1.27)
+			(end 1.33 1.27)
 			(stroke
 				(width 0.12)
@@
 		)
 		(fp_line
-			(start -1.33 1.27)
-			(end 1.33 1.27)
+			(start 1.33 1.27)
+			(end 1.33 8.95)
 			(stroke
 				(width 0.12)
@@
 		)
 		(fp_line
-			(start -1.33 1.27)
-			(end -1.33 8.95)
+			(start 0 -1.33)
+			(end 1.33 -1.33)
 			(stroke
 				(width 0.12)
@@
 		)
 		(fp_line
-			(start -1.33 8.95)
-			(end 1.33 8.95)
+			(start 1.33 -1.33)
+			(end 1.33 0)
 			(stroke
 				(width 0.12)
@@
 		)
 		(fp_line
-			(start 1.75 -1.8)
-			(end 1.75 9.4)
+			(start -1.8 9.4)
+			(end -1.8 -1.8)
 			(stroke
 				(width 0.05)
@@
 		)
 		(fp_line
-			(start -1.8 -1.8)
-			(end 1.75 -1.8)
+			(start 1.75 9.4)
+			(end -1.8 9.4)
 			(stroke
 				(width 0.05)
@@
 		)
 		(fp_line
-			(start 1.75 9.4)
-			(end -1.8 9.4)
+			(start -1.8 -1.8)
+			(end 1.75 -1.8)
 			(stroke
 				(width 0.05)
@@
 		)
 		(fp_line
-			(start -1.8 9.4)
-			(end -1.8 -1.8)
+			(start 1.75 -1.8)
+			(end 1.75 9.4)
 			(stroke
 				(width 0.05)
@@
 		)
 		(fp_line
-			(start 0.635 -1.27)
-			(end 1.27 -0.635)
+			(start -1.27 8.89)
+			(end -1.27 -1.27)
 			(stroke
 				(width 0.1)
@@
 		)
 		(fp_line
-			(start -1.27 -1.27)
-			(end 0.635 -1.27)
+			(start 1.27 8.89)
+			(end -1.27 8.89)
 			(stroke
 				(width 0.1)
@@
 		)
 		(fp_line
-			(start 1.27 8.89)
-			(end -1.27 8.89)
+			(start -1.27 -1.27)
+			(end 0.635 -1.27)
 			(stroke
 				(width 0.1)
@@
 		)
 		(fp_line
-			(start -1.27 8.89)
-			(end -1.27 -1.27)
+			(start 0.635 -1.27)
+			(end 1.27 -0.635)
 			(stroke
 				(width 0.1)
@@
 		)
 		(fp_text user "${REFERENCE}"
-			(at 0 3.81 180)
+			(at 0 3.81 0)
 			(layer "F.Fab")
 			(effects
@@
 		)
 		(pad "1" thru_hole rect
-			(at 0 0 90)
+			(at 0 0 270)
 			(size 1.7 1.7)
 			(drill 1)
@@
 		)
 		(pad "2" thru_hole circle
-			(at 0 2.54 90)
+			(at 0 2.54 270)
 			(size 1.7 1.7)
 			(drill 1)
@@
 		)
 		(pad "3" thru_hole circle
-			(at 0 5.08 90)
+			(at 0 5.08 270)
 			(size 1.7 1.7)
 			(drill 1)
@@
 		)
 		(pad "4" thru_hole circle
-			(at 0 7.62 90)
+			(at 0 7.62 270)
 			(size 1.7 1.7)
 			(drill 1)
@@
 	)
 	(segment
+		(start 188.325 90.82)
+		(end 186.08 88.575)
+		(width 0.15)
+		(layer "F.Cu")
+		(net 17)
+	)
+	(segment
+		(start 193.63 90.82)
+		(end 188.325 90.82)
+		(width 0.15)
+		(layer "F.Cu")
+		(net 17)
+	)
+	(segment
 		(start 230.22 102.38)
 		(end 230.2 102.4)
@@
 		(net 17)
 	)
+	(via
+		(at 193.63 90.82)
+		(size 0.6)
+		(drill 0.3)
+		(layers "F.Cu" "B.Cu")
+		(net 17)
+	)
 	(segment
-		(start 193.695 90.895)
-		(end 193.695 88.775)
+		(start 193.63 90.83)
+		(end 193.63 90.82)
 		(width 0.15)
 		(layer "B.Cu")
@@
 	)
 	(segment
-		(start 230.2 102.4)
-		(end 205.2 102.4)
+		(start 205.2 102.4)
+		(end 193.63 90.83)
 		(width 0.15)
 		(layer "B.Cu")
@@
 	)
 	(segment
-		(start 205.2 102.4)
-		(end 193.695 90.895)
+		(start 230.2 102.4)
+		(end 205.2 102.4)
 		(width 0.15)
 		(layer "B.Cu")
@@
 	)
 	(segment
-		(start 219.474 103.25)
-		(end 204.840412 103.25)
+		(start 220.626 103.25)
+		(end 230.2 103.25)
 		(width 0.15)
 		(layer "B.Cu")
@@
 	)
 	(segment
-		(start 230.2 103.25)
-		(end 220.626 103.25)
+		(start 220.612412 103.25)
+		(end 220.626 103.236412)
 		(width 0.15)
 		(layer "B.Cu")
@@
 	)
 	(segment
-		(start 192.69 90.06)
-		(end 191.18 88.55)
+		(start 220.626 103.236412)
+		(end 220.626 103.25)
 		(width 0.15)
 		(layer "B.Cu")
@@
 	)
 	(segment
-		(start 220.626 103.25)
-		(end 220.626 103.236412)
+		(start 219.487588 103.25)
+		(end 220.612412 103.25)
 		(width 0.15)
 		(layer "B.Cu")
@@
 	)
 	(segment
-		(start 204.840412 103.25)
-		(end 192.69 91.099588)
+		(start 188.62 88.575)
+		(end 190.905 90.86)
 		(width 0.15)
 		(layer "B.Cu")
@@
 	)
 	(segment
-		(start 220.626 103.236412)
-		(end 220.612412 103.25)
+		(start 190.905 90.86)
+		(end 192.63 90.86)
 		(width 0.15)
 		(layer "B.Cu")
@@
 	)
 	(segment
-		(start 220.612412 103.25)
+		(start 219.474 103.236412)
 		(end 219.487588 103.25)
 		(width 0.15)
@@
 	)
 	(segment
-		(start 219.487588 103.25)
-		(end 219.474 103.236412)
+		(start 192.63 90.86)
+		(end 205.02 103.25)
 		(width 0.15)
 		(layer "B.Cu")
@@
 	)
 	(segment
-		(start 219.474 103.236412)
-		(end 219.474 103.25)
+		(start 219.474 103.25)
+		(end 219.474 103.236412)
 		(width 0.15)
 		(layer "B.Cu")
@@
 	)
 	(segment
-		(start 192.69 91.099588)
-		(end 192.69 90.06)
+		(start 205.02 103.25)
+		(end 219.474 103.25)
 		(width 0.15)
 		(layer "B.Cu")
@@
 	)
 	(segment
-		(start 177.332238 72.21)
-		(end 176.93 72.21)
-		(width 0.15)
-		(layer "F.Cu")
-		(net 53)
-	)
-	(segment
-		(start 208.25 83.35)
-		(end 205.8 80.9)
+		(start 208.25 91)
+		(end 208.25 83.63)
 		(width 0.15)
 		(layer "F.Cu")
@@
 	)
 	(segment
-		(start 164.5325 72.21)
-		(end 164.505 72.2375)
+		(start 186.022238 80.9)
+		(end 177.332238 72.21)
 		(width 0.15)
 		(layer "F.Cu")
@@
 	)
 	(segment
-		(start 176.91 72.21)
-		(end 168.59 72.21)
+		(start 211.105 93.855)
+		(end 208.25 91)
 		(width 0.15)
 		(layer "F.Cu")
@@
 	)
 	(segment
-		(start 208.25 91)
-		(end 208.25 83.35)
+		(start 208.25 83.63)
+		(end 205.52 80.9)
 		(width 0.15)
 		(layer "F.Cu")
@@
 	)
 	(segment
-		(start 215 93.855)
-		(end 211.105 93.855)
+		(start 164.5325 72.21)
+		(end 164.505 72.2375)
 		(width 0.15)
 		(layer "F.Cu")
@@
 	)
 	(segment
-		(start 215 93.89)
-		(end 215 93.855)
+		(start 177.332238 72.21)
+		(end 168.59 72.21)
 		(width 0.15)
 		(layer "F.Cu")
@@
 	)
 	(segment
-		(start 205.8 80.9)
-		(end 186.022238 80.9)
+		(start 215 93.855)
+		(end 211.105 93.855)
 		(width 0.15)
 		(layer "F.Cu")
@@
 	)
 	(segment
-		(start 186.022238 80.9)
-		(end 177.332238 72.21)
+		(start 215 93.89)
+		(end 215 93.855)
 		(width 0.15)
 		(layer "F.Cu")
@@
 	)
 	(segment
-		(start 211.105 93.855)
-		(end 208.25 91)
+		(start 205.52 80.9)
+		(end 186.022238 80.9)
 		(width 0.15)
 		(layer "F.Cu")
